Commit message: avoid smallball

File: lbr_iiwa7_r800.urdf (robot description, URDF)
Before this commit: robot lbr_iiwa7_r800, 8 links, 7 joints
Links:
- added link small_ball, mass 0.01; collision sphere radius=0.01; visual sphere radius=0.01
Joints:
- added joint jointball: type revolute, parent base_link, child small_ball, origin xyz=0.2 0 1 rpy=0 0 0, axis 0 0 -1, limit lower=0 upper=0 effort=0 velocity=0
